File: KU-14194HB-REV-B-KiCad.kicad_pcb (KiCad board)
At the start: 2 copper layers, 387.7 x 180.3 mm, 149 parts, among them CN1 KEYBOARD_20PIN_MALE, CN10 LED_CONNECTOR, CN2 USER_PORT_CON, CN3 CASSETTE_PORT_CON, CN4 SERIAL_BUS_CON, CN7 POWER_CON, CN8 CONTROL_PORT, CN9 CONTROL_PORT, Q1 2SC1815, Q2 2SC1815, Q3 TP298/2SD880, Q7 2SC1815, SW1 POWER_SWITCH, U1 CIA_U1, U10 4164-2, U11 4164-2, U12 4164-2, U13 74LS257, U2 CIA_U2, U20 556, U21 4164-2, U22 4164-2, U23 4164-2, U24 4164-2, U25 74LS257, U27 7408_U27, U28 4066_U28, U29 74LS74, U30 74LS193, U31 74LS629N, U32 MC4044, U7 6510_MPU, U8 7406N, U9 4164-2, Y1 Crystal

Commit message: Tighter ram symbols. Getting closer to the end of the schematics.
Parts:
- added C17: 10uF, KU-14194HB-RevB-KiCad:CAP_ELYT_RADIAL_P2.54mm, F.Cu at (297.2, 94.0)
- added C31: .1, KU-14194HB-RevB-KiCad:CAP_P5.08mm, F.Cu at (152.4, 170.2)
- added C33: .1, KU-14194HB-RevB-KiCad:CAP_P5.08mm, F.Cu at (200.7, 170.2)
- added C4: .1, KU-14194HB-RevB-KiCad:CAP_P5.08mm, F.Cu at (91.4, 76.2)
- added C5: .1, KU-14194HB-RevB-KiCad:CAP_P5.08mm, F.Cu at (119.4, 76.2)
- added C6: .1, KU-14194HB-RevB-KiCad:CAP_P5.08mm, F.Cu at (147.3, 76.2)
- added C61: .1, KU-14194HB-RevB-KiCad:CAP_P5.08mm, F.Cu at (345.4, 154.9)
- added C63: .1, KU-14194HB-RevB-KiCad:CAP_P5.08mm, F.Cu at (363.2, 149.9)
- added C64: 10uF, KU-14194HB-RevB-KiCad:CAP_ELYT_RADIAL_P2.54mm, F.Cu at (363.2, 144.8)
- added CN6: EXPANSION_PORT, KU-14194HB-RevB-KiCad:EXPANSION_PORT, F.Cu at (307.3, 83.8)
- added FB4: FERRITE_BEAD, KU-14194HB-RevB-KiCad:FERRITE_BEAD_TH_P12.7mm, F.Cu at (243.8, 130.8)
- added L1: 2.2uH, KU-14194HB-RevB-KiCad:RESISTOR, F.Cu at (363.2, 154.9)
- added R51: 1.5K, KU-14194HB-RevB-KiCad:RESISTOR, F.Cu at (317.5, 111.8)
- added U15: 74LS139, KU-14194HB-RevB-KiCad:DIP16, F.Cu at (156.2, 156.2)
- added U17: PLA_U17, KU-14194HB-RevB-KiCad:DIP28, F.Cu at (198.1, 148.6)
- added U3: 2364A, KU-14194HB-RevB-KiCad:DIP24, F.Cu at (96.5, 95.2)
- added U4: 2364A, KU-14194HB-RevB-KiCad:DIP24, F.Cu at (121.9, 95.2)
- added U5: 2332A, KU-14194HB-RevB-KiCad:DIP24, F.Cu at (147.3, 95.2)
- C107, C108: value 10uF -> 10
Connections:
- C19 pad 1: /Sheet1/9V_UNREG -> +9V_UNREG
- C95 pad 1: /Sheet1/9V_UNREG -> +9V_UNREG
- CR4 pad 1: /Sheet1/9V_UNREG -> +9V_UNREG
- CR6 pad 2: /Sheet1/9V_UNREG -> +9V_UNREG
- RP4 pad 10: (no net) -> /Sheet5D659BBD/~DMA~
- RP4 pad 2: (no net) -> ~IRQ~
- RP4 pad 3: (no net) -> Net-(RP4-Pad3)
- RP4 pad 7: (no net) -> /Sheet5D659BBD/~GAME~
- RP4 pad 9: (no net) -> /Sheet5D659BBD/~EXROM~
- U27 pad 1: (no net) -> /Sheet5D659BBD/BA
- U27 pad 2: (no net) -> /Sheet5D659BBD/~DMA~
- U27 pad 3: (no net) -> RDY
- U27 pad 4: (no net) -> /Sheet5D659BBD/AEC
- U27 pad 5: (no net) -> /Sheet5D659BBD/~DMA~
- U27 pad 6: (no net) -> CAEC
- U8 pad 11: Net-(U8-Pad11) -> ~VA14~
- VR2 pad 1: /Sheet1/9V_UNREG -> +9V_UNREG
Routing:
- net (no net): track 7123.8 -> 3397.0 mm, vias 266 -> 156
- net /Sheet5D659BBD/BA: track 0.00 -> 416.9 mm, vias 0 -> 8
- net /Sheet5D659BBD/~ROML~: track 0.00 -> 382.6 mm, vias 0 -> 4
- net /Sheet5D659BBD/~DMA~: track 0.00 -> 346.3 mm, vias 0 -> 3
- net Net-(CN6-Pad10): track 0.00 -> 332.1 mm, vias 0 -> 3
- net Net-(CN6-Pad7): track 0.00 -> 283.6 mm, vias 0 -> 5
- net /Sheet1/9V_UNREG: track 268.7 -> 0.00 mm, vias 5 -> 0
- net +9V_UNREG: track 0.00 -> 268.7 mm, vias 0 -> 5
- net /Sheet5D659BBD/~EXROM~: track 0.00 -> 267.2 mm, vias 0 -> 8
- net /Sheet5D659BBD/~GAME~: track 0.00 -> 262.2 mm, vias 0 -> 7
- net /Sheet5D659BBD/~ROMH~: track 0.00 -> 230.5 mm, vias 0 -> 5
- net /Sheet5D659BBD/AEC: track 0.00 -> 206.2 mm, vias 0 -> 11
- net /Sheet5D659BBD/~BASIC~: track 0.00 -> 173.6 mm, vias 0 -> 2
- net /Sheet5D659BBD/~KERNAL: track 0.00 -> 156.3 mm, vias 0 -> 3
- net ~VA14~: track 210.2 -> 351.6 mm, vias 5 -> 8
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