File: KU-14194HB-REV-B-KiCad.kicad_pcb (KiCad board)
At the start: 2 copper layers, 388.6 x 180.3 mm, 219 parts, among them CN1 KEYBOARD_20PIN_MALE, CN10 LED_CONNECTOR, CN2 USER_PORT_CON, CN3 CASSETTE_PORT_CON, CN4 SERIAL_BUS_CON, CN5 AV_CONN, CN6 EXPANSION_PORT, CN7 POWER_CON, CN8 CONTROL_PORT, CN9 CONTROL_PORT, M1 MODULATOR_LONGBOARD, Q1 2SC1815, Q2 2SC1815, Q3 TP298/2SD880, Q7 2SC1815, Q8 2SC1815, SW1 POWER_SWITCH, U1 CIA_U1, U10 4164-2, U11 4164-2, U12 4164-2, U13 74LS257, U14 74LS258, U15 74LS139, U16 4066_U28, U17 PLA_U17, U18 6581, U19 VIC, U2 CIA_U2, U20 556, U21 4164-2, U22 4164-2, U23 4164-2, U24 4164-2, U25 74LS257, U26 74LS373, U27 7408_U27, U28 4066_U28, U29 74LS74, U3 2364A, U30 74LS193, U31 74LS629N, U32 MC4044, U4 2364A, U5 2332A, U6 2114, U7 6510_MPU, U8 7406N, U9 4164-2, Y1 Crystal

Commit message: update soldermask with V1.1
Other:
- board text added: "Replica 1.1 by BWACK 2019"
- board text removed: "Replica 1.0 by BWACK 2019"
Changed lines of the file:
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@@
     (36 B.SilkS user)
     (37 F.SilkS user)
-    (38 B.Mask user hide)
-    (39 F.Mask user hide)
+    (38 B.Mask user)
+    (39 F.Mask user)
     (40 Dwgs.User user)
     (41 Cmts.User user)
@@
   (gr_line (start 80.0735 56.515) (end 81.3435 56.515) (layer Edge.Cuts) (width 0.1))
   (gr_line (start 80.0735 47.3075) (end 80.0735 56.515) (layer Edge.Cuts) (width 0.1))
-  (gr_text "Replica 1.0 by BWACK 2019" (at 354.584 223.0755) (layer F.Mask)
+  (gr_text "Replica 1.1 by BWACK 2019" (at 354.584 223.0755) (layer F.Mask)
     (effects (font (size 2 2) (thickness 0.3)))
   )

Commit message: Rev 1.2
Added missing C14
Parts:
- added C14: 10uF, KU-14194HB-RevB-KiCad:CAP_ELYT_RADIAL_P2.54mm, F.Cu at (55.9, 180.3)
Routing:
- net Earth: vias 98 -> 97
Changed lines of the file:
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@@
-(kicad_pcb (version 20171130) (host pcbnew 5.1.4-e60b266~84~ubuntu16.04.1)
+(kicad_pcb (version 20171130) (host pcbnew "(5.1.4)-1")
   (general
     (thickness 1.6)
-    (drawings 11857)
-    (tracks 7004)
+    (drawings 11849)
+    (tracks 7003)
     (zones 0)
-    (modules 219)
+    (modules 220)
     (nets 253)
   )
@@
   (title_block
     (title "C64 Motherboard KU-14194HB")
-    (date 2019-10-15)
-    (rev 1.1)
+    (date 2019-11-10)
+    (rev 1.2)
     (company "Commodore 1982")
     (comment 1 "layout retraced and schematics drawn by bwack 2019")
@@
       (net 245 "Net-(CN5-Pad7)"))
   )
+  (module KU-14194HB-RevB-KiCad:CAP_ELYT_RADIAL_P2.54mm (layer F.Cu)
+    (at 55.88 180.34)
+    (fp_text reference C14 (at 0 1.27) (layer F.SilkS) hide
+      (effects (font (size 1 1) (thickness 0.15)))
+    )
+    (fp_text value 10uF (at 0 1.27) (layer F.Fab)
+      (effects (font (size 1 1) (thickness 0.15)))
+    )
+    (pad 1 thru_hole rect (at 0 0) (size 1.8 1.8) (drill 1.1) (layers *.Cu *.Mask)
+      (net 1 +5V))
+    (pad 2 thru_hole circle (at 2.54 0) (size 1.8 1.8) (drill 1.1) (layers *.Cu *.Mask)
+      (net 2 Earth))
+    (model "C:/Program Files/KiCad/share/kicad/modules/Capacitor_THT.pretty/C_Axial_L12.0mm_D8.5mm_P20.00mm_Horizontal.kicad_mod"
+      (at (xyz 0 0 0))
+      (scale (xyz 1 1 1))
+      (rotate (xyz 0 0 0))
+    )
+    (model ${KISYS3DMOD}/Capacitor_THT.3dshapes/C_Radial_D6.3mm_H11.0mm_P2.50mm.wrl
+      (at (xyz 0 0 0))
+      (scale (xyz 1 1 1))
+      (rotate (xyz 0 0 0))
+    )
+  )
   (gr_line (start 82.296 46.355) (end 85.4075 46.355) (layer Edge.Cuts) (width 0.1))
   (gr_line (start 80.0735 47.3075) (end 79.121 46.355) (layer Edge.Cuts) (width 0.1))
@@
   (gr_line (start 292.1 132.08) (end 292.1 132.08) (layer B.Mask) (width 2.2))
   (gr_line (start 292.1 139.7) (end 292.1 139.7) (layer B.Mask) (width 2.2))
-  (gr_line (start 58.42 180.34) (end 58.42 180.34) (layer B.Mask) (width 2.7))
-  (gr_poly (pts (xy 57.23 181.69) (xy 54.53 181.69) (xy 54.53 178.99) (xy 57.23 178.99)) (layer B.Mask) (width 0))
   (gr_line (start 83.82 71.12) (end 83.82 71.12) (layer B.Mask) (width 2.6))
   (gr_line (start 83.82 76.2) (end 83.82 76.2) (layer B.Mask) (width 2.6))
@@
   (gr_line (start 292.1 132.08) (end 292.1 132.08) (layer F.Mask) (width 2.2))
   (gr_line (start 292.1 139.7) (end 292.1 139.7) (layer F.Mask) (width 2.2))
-  (gr_line (start 58.42 180.34) (end 58.42 180.34) (layer F.Mask) (width 2.7))
-  (gr_poly (pts (xy 57.23 181.69) (xy 54.53 181.69) (xy 54.53 178.99) (xy 57.23 178.99)) (layer F.Mask) (width 0))
   (gr_line (start 83.82 71.12) (end 83.82 71.12) (layer F.Mask) (width 2.6))
   (gr_line (start 83.82 76.2) (end 83.82 76.2) (layer F.Mask) (width 2.6))
@@
   (gr_line (start 63.5 147.32) (end 63.5 147.32) (layer Dwgs.User) (width 1.09982))
   (gr_line (start 55.88 175.26) (end 55.88 175.26) (layer Dwgs.User) (width 1.09982))
-  (gr_line (start 55.88 180.34) (end 55.88 180.34) (layer Dwgs.User) (width 1.09982))
-  (gr_line (start 58.42 180.34) (end 58.42 180.34) (layer Dwgs.User) (width 1.09982))
   (gr_line (start 58.42 185.42) (end 58.42 185.42) (layer Dwgs.User) (width 1.09982))
   (gr_line (start 63.5 185.42) (end 63.5 185.42) (layer Dwgs.User) (width 1.09982))
@@
   (gr_line (start 48.26 96.52) (end 48.26 96.52) (layer Dwgs.User) (width 1.09982))
   (gr_line (start 272.288 106.299) (end 272.288 106.299) (layer Dwgs.User) (width 1.19888))
-  (gr_poly (pts (xy 56.93 181.39) (xy 54.83 181.39) (xy 54.83 179.29) (xy 56.93 179.29)) (layer B.Cu) (width 0))
   (gr_poly (pts (xy 392.21 206.79) (xy 390.11 206.79) (xy 390.11 204.69) (xy 392.21 204.69)) (layer B.Cu) (width 0))
   (gr_poly (pts (xy 395.19 181.83) (xy 397.29 181.83) (xy 397.29 183.93) (xy 395.19 183.93)) (layer B.Cu) (width 0))
@@
   (gr_poly (pts (xy 236.5566 101.5109) (xy 236.5566 99.328) (xy 236.5412 99.3126) (xy 236.987 99.474) (xy 237.3176 99.72) (xy 237.5097 100.0505) (xy 237.6173 100.6193) (xy 237.3944 101.0343) (xy 237.1177 101.3802) (xy 236.8333 101.5263) (xy 236.5874 101.5416)) (layer B.Cu) (width 0))
   (gr_poly (pts (xy 19.685 75.2475) (xy 24.13 75.2475) (xy 24.13 76.835) (xy 20.955 80.645) (xy 19.685 80.645)) (layer F.Cu) (width 0))
-  (gr_poly (pts (xy 56.93 181.39) (xy 54.83 181.39) (xy 54.83 179.29) (xy 56.93 179.29)) (layer F.Cu) (width 0))
   (segment (start 232.2164 106.2365) (end 232.0919 106.392) (width 0.222) (layer B.Cu) (net 0))
   (segment (start 232.0919 106.392) (end 231.843 106.4698) (width 0.222) (layer B.Cu) (net 0))
@@
   (via (at 91.44 137.16) (size 1.6) (drill 1.1) (layers F.Cu B.Cu) (net 1))
   (via (at 101.6 137.16) (size 1.6) (drill 1.1) (layers F.Cu B.Cu) (net 1))
-  (via (at 76.2 76.2) (size 1.6) (drill 1.1) (layers F.Cu B.Cu) (net 1) (status 1000000))
+  (via (at 76.2 76.2) (size 1.6) (drill 1.1) (layers F.Cu B.Cu) (net 1))
   (via (at 81.28 76.2) (size 1.6) (drill 1.1) (layers F.Cu B.Cu) (net 1))
   (via (at 20.32 78.74) (size 1.6) (drill 1.1) (layers F.Cu B.Cu) (net 1))
@@
   (segment (start 222.2052 163.4276) (end 222.3288 136.108) (width 0.3) (layer B.Cu) (net 2))
   (segment (start 222.3288 136.108) (end 220.98 134.62) (width 0.3) (layer B.Cu) (net 2))
-  (via (at 58.42 180.34) (size 2.1) (drill 1.1) (layers F.Cu B.Cu) (net 2))
   (segment (start 381 63.5) (end 381 68.58) (width 1.3) (layer B.Cu) (net 2))
   (segment (start 360.68 78.74) (end 360.68 73.66) (width 1.3) (layer B.Cu) (net 2))

Commit message: Update V1.3
See readme
Parts:
- C36: value .1 -> 20pF
- C86: value ? -> 82pF
Connections:
- R22 pad 1: Net-(R22-Pad1) -> Net-(C87-Pad1)
Routing:
- net Net-(C87-Pad1): track 11.2 -> 14.8 mm
Other:
- board text added: "Replica 1.3 by BWACK 2019"
- board text removed: "Replica 1.1 by BWACK 2019"

Commit message: Rev 1.4. See Readme
Parts:
- moved CN6 0.94 mm to (306.4, 83.8)
Routing:
- net PHI2: track 596.8 -> 597.9 mm
- net /Sheet5D659BBD/~ROML~: track 382.6 -> 383.5 mm
- net A11: track 615.7 -> 614.7 mm
- net /Sheet5D659BBD/BA: track 416.9 -> 417.8 mm
- net A10: track 674.8 -> 673.9 mm
- net A9: track 675.7 -> 674.9 mm
- net ~NMI~: track 507.0 -> 507.5 mm
Other:
- board size 388.6 x 180.3 mm -> 390.2 x 180.3 mm
- board text added: "Replica 1.4 by BWACK 2019"
- board text removed: "Replica 1.3 by BWACK 2019"
