File: file5D659BBD.sch (KiCad schematic (older format))
At the start: 89 parts, among them CN5 AV_CONN, CN6 EXPANSION_PORT, J1212 Conn_01x04, J1213 Conn_01x04, Q8 2SC1815, U10 4164-2, U11 4164-2, U12 4164-2, U13 74LS257, U14 74LS258, U15 74LS139, U16 4066_U28, U17 PLA_U17, U18 6581, U19 VIC, U21 4164-2, U22 4164-2, U23 4164-2, U24 4164-2, U25 74LS257, U26 74LS373, U27 7408_U27, U3 2364A, U4 2364A, U5 2332A, U6 2114, U8 7406N, U9 4164-2

Commit message: Replica 1.0
Parts:
- removed J1212, J1213: Conn_01x04, symbol Connector_Generic:Conn_01x04
- added M1: MODULATOR_LONGBOARD, KU-14194HB-RevB-KiCad:MODULATOR_PORT_LONGBOARD, symbol KU-schematics-library:MODULATOR_LONGBOARD
- U6: footprint (none) -> KU-14194HB-RevB-KiCad:DIP18
Connections:
- net +9V_UNREG: now also M1.1 (9V)
- net AUDIO_OUT: now also M1.4 (AUDIO)
- net CHROMA: now also M1.3 (CHR); no longer CN5.6
- net GR\~W~: now also U17.13 (F4)
- net LUMA: now also M1.2 (LUM); no longer CN5.1
- net VA4: now also U17.20 (I15)
- net VA5: now also U17.21 (I14)
- net ~CHAREN~: no longer U14.2 (A0), U17.5 (I4)
- net COMP renamed COMP_O
- net COMP_O: now also M1.5 (COMP)
- new net CHROMA_O: CN5.6, M1.7 (CHR)
- new net LUMA_O: CN5.1, M1.6 (LUM)
- new net ~VA14~: U14.2 (A0), U17.5 (I4)
Other:
- note removed: "RF MODULATOR"
Changed lines of the file:
@@
 Sheet 3 3
 Title "C64 Motherboard KU-14194HB"
-Date "2019-09-29"
-Rev ""
+Date "2019-10-05"
+Rev "1.0"
 Comp "Commodore 1982"
 Comment1 "Retraced and schematics by bwack 2019"
@@
 Connection ~ 1100 7650
 Wire Wire Line
-	1100 7250 1100 7650
-Wire Wire Line
 	1000 7250 1100 7250
 Text Label 3450 7550 0    50   ~ 0
@@
 	4700 6800 6050 6800
 Wire Wire Line
-	7400 5250 7400 8950
-Wire Wire Line
-	7500 5250 7500 9050
-Wire Wire Line
 	4600 7350 5100 7350
 Wire Wire Line
@@
 	1600 800  1600 6000
 Wire Wire Line
-	1100 700  1100 7250
-Connection ~ 1100 7250
-Wire Wire Line
 	1100 7250 1200 7250
 $Comp
@@
 F 0 "U6" H 10500 6250 79  0000 L CNN
 F 1 "2114" H 10450 6100 55  0000 L CNN
-F 2 "" H 10500 5600 39  0001 C CNN
+F 2 "KU-14194HB-RevB-KiCad:DIP18" H 10500 5600 39  0001 C CNN
 F 3 "" H 10500 5600 39  0001 C CNN
 	1    10500 5800
@@
 	8150 5200 8150 5600
 Wire Wire Line
-	8250 5200 8250 5600
+	8250 5200 8250 5550
 Wire Wire Line
-	8350 5200 8350 5600
+	8350 5200 8350 5500
 Wire Wire Line
 	8450 5200 8450 5600
@@
 AEC
 Wire Wire Line
-	4650 7650 10550 7650
+	4600 7650 10550 7650
 Wire Wire Line
 	10550 7650 10550 6600
@@
 Connection ~ 12800 1400
 Wire Wire Line
-	13300 1400 13700 1400
+	13300 1400 13600 1400
 $Comp
 L Device:C_Small C54
@@
 	13500 1900 13300 1900
 Connection ~ 13300 1900
-Text Label 13700 1400 2    50   ~ 0
-CAN+5V
 $Comp
 L KU-14194HB-REV-B-KiCad-rescue:GND_SMALL-power #U0218
@@
 Text Label 12350 2450 0    50   ~ 0
 +9V_UNREG
-$Comp
-L Connector_Generic:Conn_01x04 J1212
-U 1 1 5D9C771C
-P 13700 2950
-F 0 "J1212" H 13780 2896 50  0001 L CNN
-F 1 "Conn_01x04" H 13780 2851 50  0001 L CNN
-F 2 "" H 13700 2950 50  0001 C CNN
-F 3 "~" H 13700 2950 50  0001 C CNN
-	1    13700 2950
-	1    0    0    -1
-$EndComp
-Wire Notes Line
-	13450 2700 15050 2700
-Wire Notes Line
-	15050 2700 15050 3300
-Wire Notes Line
-	15050 3300 13450 3300
-Wire Notes Line
-	13450 3300 13450 2700
-Text Notes 13800 3050 0    79   ~ 0
-RF MODULATOR
 Wire Wire Line
 	13500 2850 13300 2450
@@
 	1    0    0    -1
 $EndComp
-Text Label 15200 2850 0    50   ~ 0
-COMP
-Text Label 15200 2950 0    50   ~ 0
-LUMA
-Text Label 15200 3050 0    50   ~ 0
-CHROMA
+Text Label 15150 2850 0    50   ~ 0
+COMP_O
+Text Label 15150 2950 0    50   ~ 0
+LUMA_O
+Text Label 15150 3050 0    50   ~ 0
+CHROMA_O
 Text Notes 15900 6150 1    79   Italic 0
 AUDIO/VIDEO (8 PIN FEMALE DIN)
@@
 Wire Wire Line
 	15550 2850 15000 2850
-$Comp
-L Connector_Generic:Conn_01x04 J1213
-U 1 1 5D9C8179
-P 14800 2950
-F 0 "J1213" H 14718 2617 50  0001 C CNN
-F 1 "Conn_01x04" H 14718 2616 50  0001 C CNN
-F 2 "" H 14800 2950 50  0001 C CNN
-F 3 "~" H 14800 2950 50  0001 C CNN
-	1    14800 2950
-	-1   0    0    -1
-$EndComp
 Wire Wire Line
 	14900 5800 14900 5950
@@
 	1    0    0    -1
 $EndComp
+Text GLabel 13600 1400 2    50   Input ~ 0
+CAN+5V
+Text Label 3650 8650 0    28   ~ 0
+VA5
+Text Label 3750 8750 0    28   ~ 0
+VA4
+Wire Wire Line
+	8250 5550 7500 5550
+Connection ~ 8250 5550
+Wire Wire Line
+	8250 5550 8250 5600
+Wire Wire Line
+	7500 5550 7500 9050
+Wire Wire Line
+	8350 5500 7400 5500
+Connection ~ 8350 5500
+Wire Wire Line
+	8350 5500 8350 5600
+Wire Wire Line
+	7400 5500 7400 8950
+$Comp
+L KU-schematics-library:MODULATOR_LONGBOARD M1
+U 1 1 5DC37670
+P 14050 2950
+F 0 "M1" H 14050 2950 39  0001 C CNN
+F 1 "MODULATOR_LONGBOARD" H 14050 2950 39  0001 C CNN
+F 2 "KU-14194HB-RevB-KiCad:MODULATOR_PORT_LONGBOARD" H 14050 2950 39  0001 C CNN
+F 3 "" H 14050 2950 39  0001 C CNN
+	1    14050 2950
+	1    0    0    -1
+$EndComp
+Wire Wire Line
+	1100 700  1100 7650
 Wire Bus Line
 	8400 8950 8400 9150
