File: file5D659BBD.sch (KiCad schematic (older format))
At the start: 88 parts, among them CN5 AV_CONN, CN6 EXPANSION_PORT, M1 MODULATOR_LONGBOARD, Q8 2SC1815, U10 4164-2, U11 4164-2, U12 4164-2, U13 74LS257, U14 74LS258, U15 74LS139, U16 4066_U28, U17 PLA_U17, U18 6581, U19 VIC, U21 4164-2, U22 4164-2, U23 4164-2, U24 4164-2, U25 74LS257, U26 74LS373, U27 7408_U27, U3 2364A, U4 2364A, U5 2332A, U6 2114, U8 7406N, U9 4164-2

Commit message: Rev 1.2
Added missing C14
Parts:
- added C14: 10uF, KU-14194HB-RevB-KiCad:CAP_ELYT_RADIAL_P2.54mm, symbol Device:CP_Small
Connections:
- net +5V: now also C14.1
- net Earth: now also C14.2

Commit message: Update V1.3
See readme
Other:
- note added: "Y5U"
Changed lines of the file:
@@
 Sheet 3 3
 Title "C64 Motherboard KU-14194HB"
-Date "2019-11-10"
-Rev "1.2"
+Date "2019-11-12"
+Rev "1.3"
 Comp "Commodore 1982"
 Comment1 "Retraced and schematics by bwack 2019"
@@
 Wire Wire Line
 	8150 1350 7700 1350
+$Comp
+L KU-14194HB-REV-B-KiCad-rescue:GND_SMALL-power-KU-14194HB-REV-B-KiCad-rescue #U?
+U 1 1 5DE17930
+P 8150 1550
+AR Path="/5DE17930" Ref="#U?"  Part="1"
+AR Path="/5D659BBE/5DE17930" Ref="#U0242"  Part="1"
+F 0 "#U0242" H 8150 1550 50  0001 C CNN
+F 1 "GND_SMALL-power" H 8150 1550 50  0001 C CNN
+F 2 "" H 8150 1550 50  0001 C CNN
+F 3 "" H 8150 1550 50  0001 C CNN
+	1    8150 1550
+	1    0    0    -1
+$EndComp
 Wire Bus Line
 	8400 8950 8400 9150
@@
 Wire Bus Line
 	2800 4350 9300 4350
-$Comp
-L KU-14194HB-REV-B-KiCad-rescue:GND_SMALL-power-KU-14194HB-REV-B-KiCad-rescue #U?
-U 1 1 5DE17930
-P 8150 1550
-AR Path="/5DE17930" Ref="#U?"  Part="1"
-AR Path="/5D659BBE/5DE17930" Ref="#U?"  Part="1"
-F 0 "#U?" H 8150 1550 50  0001 C CNN
-F 1 "GND_SMALL-power" H 8150 1550 50  0001 C CNN
-F 2 "" H 8150 1550 50  0001 C CNN
-F 3 "" H 8150 1550 50  0001 C CNN
-	1    8150 1550
-	1    0    0    -1
-$EndComp
+Text Notes 12550 1700 0    50   ~ 0
+Y5U
 $EndSCHEMATC

Commit message: value updates
Parts:
- R31: value 180 -> 1K
Changed lines of the file:
@@
 P 2000 1000
 F 0 "R31" V 1829 937 50  0000 L CNN
-F 1 "180" V 1914 929 50  0000 L CNN
+F 1 "1K" V 1914 929 50  0000 L CNN
 F 2 "KU-14194HB-RevB-KiCad:RESISTOR" H 2000 1000 50  0001 C CNN
 F 3 "" H 2000 1000 50  0001 C CNN
@@
 	1    0    0    -1
 $EndComp
+Text Notes 12550 1700 0    50   ~ 0
+Y5U
 Wire Bus Line
 	8400 8950 8400 9150
@@
 Wire Bus Line
 	2800 4350 9300 4350
-Text Notes 12550 1700 0    50   ~ 0
-Y5U
 $EndSCHEMATC
